Commit message: Init model

File: src/rpg2020/urdf/mrobot_chassis.urdf (robot description, URDF)
Before this commit: robot mrobot_chassis, 6 links, 5 joints
Links:
- link base_link: mass None -> 2; geometry collision cylinder length=${base_link_length} radius=${base_link_radius}; visual cylinder length=${base_link_length} radius=${base_link_radius}
